File: 3-schemaElettrico/KICAD MARZO 2025 PROTOTIPO2/Leonardo_v2.0/Stepper_Motor_driver.kicad_sch (KiCad schematic)
At the start: 1 part

Commit message: done 74hc238
Parts:
- renumbered A4 to A1
Changed lines of the file:
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@@
 		(dnp no)
 		(fields_autoplaced yes)
-		(property "Reference" "#PWR?"
+		(property "Reference" "#PWR0103"
 			(at 146.05 76.2 0)
 			(effects
@@
 				)
 				(path "/0d3207ba-e51c-4f46-8c4e-e116d0062888/e19ffaaf-7dab-4afc-b5a3-8e6e67a99faf"
-					(reference "#PWR?")
+					(reference "#PWR0103")
 					(unit 1)
 				)
@@
 		(dnp no)
 		(fields_autoplaced yes)
-		(property "Reference" "#PWR?"
+		(property "Reference" "#PWR0101"
 			(at 146.05 128.27 0)
 			(effects
@@
 				)
 				(path "/0d3207ba-e51c-4f46-8c4e-e116d0062888/e19ffaaf-7dab-4afc-b5a3-8e6e67a99faf"
-					(reference "#PWR?")
+					(reference "#PWR0101")
 					(unit 1)
 				)
@@
 		(dnp no)
 		(fields_autoplaced yes)
-		(property "Reference" "#PWR?"
+		(property "Reference" "#PWR0102"
 			(at 151.13 69.85 0)
 			(effects
@@
 				)
 				(path "/0d3207ba-e51c-4f46-8c4e-e116d0062888/e19ffaaf-7dab-4afc-b5a3-8e6e67a99faf"
-					(reference "#PWR?")
+					(reference "#PWR0102")
 					(unit 1)
 				)
@@
 		(dnp no)
 		(fields_autoplaced yes)
-		(property "Reference" "A?"
+		(property "Reference" "A1"
 			(at 153.2733 76.2 0)
 			(effects
@@
 				)
 				(path "/0d3207ba-e51c-4f46-8c4e-e116d0062888/e19ffaaf-7dab-4afc-b5a3-8e6e67a99faf"
-					(reference "A?")
-					(unit 1)
-				)
+					(reference "A1")
+					(unit 1)
+				)
