File: 3-schemaElettrico/_PCB_PROTOTIPO_2_KICAD (attivo)/Leonardo_v2.0/Leonardo_v2.0.kicad_sch (KiCad schematic)
At the start: 8 parts, among them J1 Screw_Terminal_01x02, J2 Conn_01x06_Pin, J3 Conn_01x06_Pin, J4 Conn_01x04_Pin, J5 Conn_01x04_Pin, J6 Conn_01x04_Pin, J7 Conn_01x04_Pin

Commit message: ok
Other:
- sheet Microcontroller ports: added BAT_LVL, M1, M2, M3, PWM_EN; removed INGRESSO
Changed lines of the file:
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@@
+	(wire
+		(pts
+			(xy 100.33 118.11) (xy 111.76 118.11)
+		)
+		(stroke
+			(width 0)
+			(type default)
+		)
+	)
 	(wire
 		(pts
@@
 	(wire
 		(pts
+			(xy 102.87 120.65) (xy 102.87 152.4)
+		)
+		(stroke
+			(width 0)
+			(type default)
+		)
+	)
+	(wire
+		(pts
 			(xy 62.23 157.48) (xy 48.26 157.48)
 		)
@@
 	(wire
 		(pts
+			(xy 87.63 149.86) (xy 100.33 149.86)
+		)
+		(stroke
+			(width 0)
+			(type default)
+		)
+	)
+	(wire
+		(pts
 			(xy 234.95 55.88) (xy 247.65 55.88)
 		)
@@
 	(wire
 		(pts
+			(xy 111.76 120.65) (xy 102.87 120.65)
+		)
+		(stroke
+			(width 0)
+			(type default)
+		)
+	)
+	(wire
+		(pts
+			(xy 111.76 124.46) (xy 105.41 124.46)
+		)
+		(stroke
+			(width 0)
+			(type default)
+		)
+	)
+	(wire
+		(pts
 			(xy 234.95 109.22) (xy 247.65 109.22)
 		)
@@
 	(wire
 		(pts
+			(xy 97.79 115.57) (xy 97.79 147.32)
+		)
+		(stroke
+			(width 0)
+			(type default)
+		)
+	)
+	(wire
+		(pts
 			(xy 214.63 91.44) (xy 218.44 91.44)
 		)
@@
 	(wire
 		(pts
+			(xy 105.41 154.94) (xy 87.63 154.94)
+		)
+		(stroke
+			(width 0)
+			(type default)
+		)
+	)
+	(wire
+		(pts
 			(xy 234.95 111.76) (xy 247.65 111.76)
 		)
@@
 	(wire
 		(pts
+			(xy 102.87 152.4) (xy 87.63 152.4)
+		)
+		(stroke
+			(width 0)
+			(type default)
+		)
+	)
+	(wire
+		(pts
 			(xy 62.23 171.45) (xy 48.26 171.45)
 		)
@@
 	(wire
 		(pts
+			(xy 97.79 147.32) (xy 87.63 147.32)
+		)
+		(stroke
+			(width 0)
+			(type default)
+		)
+	)
+	(wire
+		(pts
 			(xy 234.95 86.36) (xy 247.65 86.36)
 		)
@@
 	(wire
 		(pts
+			(xy 100.33 149.86) (xy 100.33 118.11)
+		)
+		(stroke
+			(width 0)
+			(type default)
+		)
+	)
+	(wire
+		(pts
 			(xy 234.95 114.3) (xy 247.65 114.3)
 		)
@@
 		(pts
 			(xy 212.09 60.96) (xy 212.09 88.9)
+		)
+		(stroke
+			(width 0)
+			(type default)
+		)
+	)
+	(wire
+		(pts
+			(xy 111.76 115.57) (xy 97.79 115.57)
+		)
+		(stroke
+			(width 0)
+			(type default)
+		)
+	)
+	(wire
+		(pts
+			(xy 105.41 124.46) (xy 105.41 154.94)
 		)
 		(stroke
@@
 			)
 		)
-		(pin "INGRESSO" input
-			(at 111.76 95.25 180)
-			(effects
-				(font
-					(size 1.27 1.27)
-				)
-				(justify left)
-			)
-		)
 		(pin "DIR3" output
 			(at 168.91 96.52 0)
@@
 			)
 		)
+		(pin "M1" output
+			(at 111.76 115.57 180)
+			(effects
+				(font
+					(size 1.27 1.27)
+				)
+				(justify left)
+			)
+		)
+		(pin "M2" output
+			(at 111.76 118.11 180)
+			(effects
+				(font
+					(size 1.27 1.27)
+				)
+				(justify left)
+			)
+		)
+		(pin "M3" output
+			(at 111.76 120.65 180)
+			(effects
+				(font
+					(size 1.27 1.27)
+				)
+				(justify left)
+			)
+		)
+		(pin "PWM_EN" output
+			(at 111.76 124.46 180)
+			(effects
+				(font
+					(size 1.27 1.27)
+				)
+				(justify left)
+			)
+		)
+		(pin "BAT_LVL" output
+			(at 111.76 86.36 180)
+			(effects
+				(font
+					(size 1.27 1.27)
+				)
+				(justify left)
+			)
+		)
