File: 3-schemaElettrico/_PCB_PROTOTIPO_2_KICAD (attivo)/Leonardo_v2.0/untitled.kicad_sch (KiCad schematic)
At the start: 0 parts

Commit message: ok
Changed lines of the file:
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@@
+		)
+	)
+	(hierarchical_label "M1"
+		(shape output)
+		(at 162.56 55.88 0)
+		(effects
+			(font
+				(size 1.27 1.27)
+			)
+			(justify left)
 		)
 	)
@@
 		)
 	)
+	(hierarchical_label "M2"
+		(shape output)
+		(at 162.56 59.69 0)
+		(effects
+			(font
+				(size 1.27 1.27)
+			)
+			(justify left)
+		)
+	)
+	(hierarchical_label "BAT_LVL"
+		(shape output)
+		(at 102.87 57.15 0)
+		(effects
+			(font
+				(size 1.27 1.27)
+			)
+			(justify left)
+		)
+	)
+	(hierarchical_label "M3"
+		(shape output)
+		(at 162.56 63.5 0)
+		(effects
+			(font
+				(size 1.27 1.27)
+			)
+			(justify left)
+		)
+	)
 	(hierarchical_label "DIR4"
 		(shape output)
@@
 		(effects
 			(font
+				(size 1.27 1.27)
+			)
+			(justify left)
+		)
+	)
+	(hierarchical_label "PWM_EN"
+		(shape output)
+		(at 162.56 50.8 0)
+		(effects
+			(font
