File: 3-schemaElettrico/_PCB_PROTOTIPO_2_KICAD (attivo)/Leonardo_v2.0/Leonardo_v2.0.kicad_pcb (KiCad board)
At the start: 2 copper layers, 0 parts

Commit message: ok
Parts:
- added A1: Pololu_Breakout_A4988, Module:Pololu_Breakout-16_15.2x20.3mm, F.Cu at (127.3, 93.2)
- added A2: Pololu_Breakout_A4988, Module:Pololu_Breakout-16_15.2x20.3mm, F.Cu at (127.3, 69.3)
- added A3: Pololu_Breakout_A4988, Module:Pololu_Breakout-16_15.2x20.3mm, F.Cu at (108.5, 93.2)
- added A4: Pololu_Breakout_A4988, Module:Pololu_Breakout-16_15.2x20.3mm, F.Cu at (108.5, 69.3)
- added Q1: BC817, Package_TO_SOT_SMD:SOT-23, F.Cu at (146.5, 93.6)
