File: 3-schemaElettrico/_PCB_PROTOTIPO_2_KICAD (attivo)/Leonardo_v2.0/Leonardo_v2.0.kicad_pcb (KiCad board)
At the start: 2 copper layers, 5 parts, among them Q1 BC817

Commit message: OK
Parts:
- added C1: 1uF, Capacitor_SMD:C_0805_2012Metric_Pad1.18x1.45mm_HandSolder, F.Cu at (75.2, 44.7)
- added D1: LED, LED_THT:LED_D3.0mm_FlatTop, F.Cu at (68.6, 45.9)
- added J1: Screw_Terminal_01x02, TerminalBlock_Phoenix:TerminalBlock_Phoenix_MKDS-1,5-2_1x02_P5.00mm_Horizontal, F.Cu at (24.1, 37.3)
- added J10: Screw_Terminal_01x02, TerminalBlock_Phoenix:TerminalBlock_Phoenix_MKDS-1,5-2_1x02_P5.00mm_Horizontal, F.Cu at (104.7, 23.0)
- added J11: Screw_Terminal_01x02, TerminalBlock_Phoenix:TerminalBlock_Phoenix_MKDS-1,5-2_1x02_P5.00mm_Horizontal, F.Cu at (119.1, 23.4)
- added J13: Conn_02x03_Odd_Even, Connector_PinHeader_2.54mm:PinHeader_2x03_P2.54mm_Vertical, F.Cu at (22.9, 94.4)
- added J2: Conn_01x06_Pin, Connector_PinHeader_2.54mm:PinHeader_1x06_P2.54mm_Vertical, F.Cu at (122.2, 34.2)
- added J3: Conn_01x06_Pin, Connector_PinHeader_2.54mm:PinHeader_1x06_P2.54mm_Vertical, F.Cu at (122.2, 50.9)
- added J4: Conn_01x04_Pin, Connector_PinHeader_2.54mm:PinHeader_1x04_P2.54mm_Vertical, F.Cu at (221.6, 27.4)
- added J5: Conn_01x04_Pin, Connector_PinHeader_2.54mm:PinHeader_1x04_P2.54mm_Vertical, F.Cu at (221.6, 50.5)
- added J6: Conn_01x04_Pin, Connector_PinHeader_2.54mm:PinHeader_1x04_P2.54mm_Vertical, F.Cu at (221.6, 73.5)
- added J7: Conn_01x04_Pin, Connector_PinHeader_2.54mm:PinHeader_1x04_P2.54mm_Vertical, F.Cu at (221.6, 96.5)
- added J8: Screw_Terminal_01x02, TerminalBlock_Phoenix:TerminalBlock_Phoenix_MKDS-1,5-2_1x02_P5.00mm_Horizontal, F.Cu at (36.2, 37.3)
- added J9: Screw_Terminal_01x02, TerminalBlock_Phoenix:TerminalBlock_Phoenix_MKDS-1,5-2_1x02_P5.00mm_Horizontal, F.Cu at (82.1, 26.4)
- added LS1: Speaker, Buzzer_Beeper:Buzzer_TDK_PS1240P02BT_D12.2mm_H6.5mm, F.Cu at (57.6, 50.1)
- added R1: 10K, Resistor_SMD:R_0805_2012Metric, F.Cu at (50.7, 44.7)
- added R2: 300K, Resistor_SMD:R_0805_2012Metric, F.Cu at (50.7, 47.6)
- added R3: R_US, Resistor_SMD:R_0805_2012Metric, F.Cu at (50.7, 50.6)
- added R4: R_US, Resistor_SMD:R_0805_2012Metric, F.Cu at (50.7, 53.5)
- added R5: R_US, Resistor_SMD:R_0805_2012Metric, F.Cu at (50.7, 56.5)
- added R6: 10K, Resistor_SMD:R_0805_2012Metric, F.Cu at (30.0, 93.5)
- added R7: 10K, Resistor_SMD:R_0805_2012Metric, F.Cu at (30.0, 96.5)
- added R8: 10K, Resistor_SMD:R_0805_2012Metric, F.Cu at (30.0, 99.4)
- added U1: ~, ESP32_NODEMCU:DIP-38_1000_ELL, F.Cu at (169.4, 49.8)
- Q1: footprint Package_TO_SOT_SMD:SOT-23 -> Package_TO_SOT_SMD:SOT-23-3
- moved A4 109.7 mm to (213.3, 101.6), turned to 180 degrees
- moved A3 105.9 mm to (213.3, 78.5), turned to 180 degrees
- moved A1 105.3 mm to (213.3, 32.5), turned to 180 degrees
- moved A2 87.1 mm to (213.3, 55.5), turned to 180 degrees
- moved Q1 42.8 mm to (126.5, 55.8)

Commit message: ok
Parts:
- added C2: 1000 uF, Capacitor_THT:CP_Radial_D10.0mm_P5.00mm, F.Cu at (189.5, 9.71)
- added C3: 1000 uF, Capacitor_THT:CP_Radial_D10.0mm_P5.00mm, F.Cu at (189.5, 33.3)
- added D2: D_Schottky, Diode_THT:D_5KPW_P12.70mm_Horizontal, F.Cu at (59.9, 84.2)
- added F1: Fuse, Fuse:Fuse_1812_4532Metric_Pad1.30x3.40mm_HandSolder, F.Cu at (82.0, 74.6)
- added U2: DC_DC_small, DC_DC_LM2596_small:DC_DC_LM2596_small, F.Cu at (157.9, 12.3)
- added U3: DC_DC_small, DC_DC_LM2596_small:DC_DC_LM2596_small, F.Cu at (157.9, 36.5)
- R5: value R_US -> 220
- moved J1 97.1 mm to (67.6, 124.1), turned to -90 degrees
- moved LS1 96.1 mm to (144.2, 91.7)
- moved J10 79.8 mm to (25.0, 18.8)
- moved J11 79.8 mm to (39.4, 19.2)
- moved Q1 31.7 mm to (139.9, 84.4)
- moved J2 31.7 mm to (135.6, 62.9)
- moved J3 31.7 mm to (135.6, 79.6)
- moved U1 29.5 mm to (183.8, 75.6)
- moved A2 11.0 mm to (222.9, 50.1)
- moved A3 11.0 mm to (222.9, 73.2)
- moved A4 11.0 mm to (222.9, 96.2)
- moved J4 11.0 mm to (231.2, 22.0)
- moved J5 11.0 mm to (231.2, 45.1)
- moved J6 11.0 mm to (231.2, 68.1)
- moved J7 11.0 mm to (231.2, 91.1)
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Connections:
- A1 pad 10: /Microcontroller/M1 -> /Microcontroller/DIR2
- A1 pad 11: /Microcontroller/M2 -> /Microcontroller/DIR3
- A2 pad 10: /Microcontroller/M1 -> /Microcontroller/DIR2
- A2 pad 11: /Microcontroller/M2 -> /Microcontroller/DIR3
- A2 pad 15: /Microcontroller/STP2 -> /Microcontroller/DIR3
- A3 pad 10: /Microcontroller/M1 -> /Microcontroller/DIR2
- A3 pad 11: /Microcontroller/M2 -> /Microcontroller/DIR3
- A3 pad 15: /Microcontroller/STP3 -> /Microcontroller/DIR2
- A4 pad 10: /Microcontroller/M1 -> /Microcontroller/DIR2
- A4 pad 11: /Microcontroller/M2 -> /Microcontroller/DIR3
- J1 pad 2: +12V -> GND
- J13 pad 4: /Microcontroller/M2 -> /Microcontroller/DIR3
- J13 pad 6: /Microcontroller/M1 -> /Microcontroller/DIR2
- R1 pad 1: Net-(J1-Pin_1) -> +BATT
- R7 pad 1: /Microcontroller/M2 -> /Microcontroller/DIR3
- R8 pad 1: /Microcontroller/M1 -> /Microcontroller/DIR2
- U1 pad 25: /Microcontroller/STP3 -> /Microcontroller/DIR2
- U1 pad 27: /Microcontroller/STP2 -> /Microcontroller/DIR3

Commit message: ok
Parts:
- removed C1: 1uF, Capacitor_SMD:C_0805_2012Metric_Pad1.18x1.45mm_HandSolder
- removed C2, C3: 1000 uF, Capacitor_THT:CP_Radial_D10.0mm_P5.00mm
- removed D1: LED, LED_THT:LED_D3.0mm_FlatTop
- removed D2: D_Schottky, Diode_THT:D_5KPW_P12.70mm_Horizontal
- removed F1: Fuse, Fuse:Fuse_1812_4532Metric_Pad1.30x3.40mm_HandSolder
- removed J11: Screw_Terminal_01x02, TerminalBlock_Phoenix:TerminalBlock_Phoenix_MKDS-1,5-2_1x02_P5.00mm_Horizontal
- removed LS1: Speaker, Buzzer_Beeper:Buzzer_TDK_PS1240P02BT_D12.2mm_H6.5mm
- removed Q1: BC817, Package_TO_SOT_SMD:SOT-23-3
- removed R5: 220, Resistor_SMD:R_0805_2012Metric
- removed U2, U3: DC_DC_small, DC_DC_LM2596_small:DC_DC_LM2596_small
- R2: value 300K -> 10K
- R3, R4: value R_US -> 10K
- moved J1 161.7 mm to (206.0, 40.3), turned to 0 degrees
- moved J8 157.8 mm to (194.0, 40.3)
- moved R1 157.8 mm to (208.5, 47.2)
- moved J10 147.1 mm to (170.5, 40.2)
- moved R2 145.8 mm to (196.5, 46.7)
- moved R3 133.3 mm to (184.0, 46.7)
- moved R6 128.5 mm to (158.4, 87.0)
- moved R7 128.5 mm to (158.4, 89.9)
- moved R8 128.5 mm to (158.4, 92.9)
- moved J13 127.7 mm to (150.5, 87.5)
- moved R4 122.5 mm to (173.0, 46.7)
- moved J9 100.8 mm to (182.0, 40.2)
- moved A2 61.9 mm to (181.3, 95.9)
- moved J5 61.9 mm to (189.6, 90.9)
- moved A1 61.9 mm to (181.3, 72.9)
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Connections:
- A1 pad 10: /Microcontroller/DIR2 -> /Stepper_Motor_driver/MS1
- A1 pad 11: /Microcontroller/DIR3 -> /Stepper_Motor_driver/MS2
- A1 pad 12: /Microcontroller/M3 -> /Stepper_Motor_driver/MS3
- A2 pad 10: /Microcontroller/DIR2 -> /Stepper_Motor_driver/MS1
- A2 pad 11: /Microcontroller/DIR3 -> /Stepper_Motor_driver/MS2
- A2 pad 12: /Microcontroller/M3 -> /Stepper_Motor_driver/MS3
- A2 pad 15: /Microcontroller/DIR3 -> /Microcontroller/STP2
- A3 pad 10: /Microcontroller/DIR2 -> /Stepper_Motor_driver/MS1
- A3 pad 11: /Microcontroller/DIR3 -> /Stepper_Motor_driver/MS2
- A3 pad 12: /Microcontroller/M3 -> /Stepper_Motor_driver/MS3
- A3 pad 15: /Microcontroller/DIR2 -> /Microcontroller/STP3
- A4 pad 10: /Microcontroller/DIR2 -> /Stepper_Motor_driver/MS1
- A4 pad 11: /Microcontroller/DIR3 -> /Stepper_Motor_driver/MS2
- A4 pad 12: /Microcontroller/M3 -> /Stepper_Motor_driver/MS3
- J1 pad 1: Net-(J1-Pin_1) -> /Microcontroller/FC1
- J10 pad 1: unconnected-(J10-Pin_1-Pad1) -> /Microcontroller/FC4
- J10 pad 2: unconnected-(J10-Pin_2-Pad2) -> GND
- J13 pad 2: /Microcontroller/M3 -> /Stepper_Motor_driver/MS1
- J13 pad 4: /Microcontroller/DIR3 -> /Stepper_Motor_driver/MS2
- J13 pad 6: /Microcontroller/DIR2 -> /Stepper_Motor_driver/MS3
- J8 pad 1: +3V3 -> /Microcontroller/FC2
- J8 pad 2: +5V -> GND
- J9 pad 1: GND -> /Microcontroller/FC3
- R1 pad 1: +BATT -> /Microcontroller/FC1
- R1 pad 2: /Microcontroller/BAT_LVL -> +3.3V
- R2 pad 1: /Microcontroller/BAT_LVL -> /Microcontroller/FC2
- R2 pad 2: GND -> +3.3V
- R3 pad 1: Net-(LS1-Pad2) -> /Microcontroller/FC3
- R3 pad 2: Net-(Q1-C) -> +3.3V
- R4 pad 1: /Microcontroller/buzzer -> /Microcontroller/FC4
- R4 pad 2: Net-(Q1-B) -> +3.3V
- R6 pad 1: /Microcontroller/M3 -> /Stepper_Motor_driver/MS1
- R7 pad 1: /Microcontroller/DIR3 -> /Stepper_Motor_driver/MS2
- R8 pad 1: /Microcontroller/DIR2 -> /Stepper_Motor_driver/MS3
- U1 pad 10: /Microcontroller/M1D -> /Microcontroller/PWM_EN_2
- U1 pad 23: /Microcontroller/STP4 -> /Microcontroller/DIR4
- U1 pad 24: /Microcontroller/DIR4 -> /Microcontroller/STP4
- U1 pad 25: /Microcontroller/DIR2 -> /Microcontroller/DIR3
- U1 pad 26: /Microcontroller/DIR3 -> /Microcontroller/STP3
- U1 pad 27: /Microcontroller/DIR3 -> /Microcontroller/DIR2
- U1 pad 28: /Microcontroller/DIR2 -> /Microcontroller/STP2
- U1 pad 29: /Microcontroller/STP1 -> /Microcontroller/DIR1
- U1 pad 30: /Microcontroller/DIR1 -> /Microcontroller/STP1
- U1 pad 31: /Microcontroller/buzzer -> /Microcontroller/FC1
- U1 pad 33: /Microcontroller/LED -> /Microcontroller/FC2
- U1 pad 36: /Microcontroller/PWM_EN_2 -> /Microcontroller/FC3
- U1 pad 37: /Microcontroller/PWM_EN_1 -> /Microcontroller/FC4
- U1 pad 5: unconnected-(U1-G34-Pad5) -> /Microcontroller/M1A
- U1 pad 6: /Microcontroller/BAT_LVL -> /Microcontroller/M1B
- U1 pad 7: /Microcontroller/M1A -> /Microcontroller/M1C
- U1 pad 8: /Microcontroller/M1B -> /Microcontroller/M1D
- U1 pad 9: /Microcontroller/M1C -> /Microcontroller/PWM_EN_1
