File: 3-schemaElettrico/_PCB_PROTOTIPO_2_KICAD (attivo)/Leonardo_v2.0/Stepper_Motor_driver.kicad_sch (KiCad schematic)
At the start: 1 part

Commit message: OK
Changed lines of the file:
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@@
 	(wire
 		(pts
-			(xy 114.3 100.33) (xy 116.84 100.33)
+			(xy 104.14 99.06) (xy 135.89 99.06)
 		)
 		(stroke
@@
 	(wire
 		(pts
-			(xy 116.84 99.06) (xy 135.89 99.06)
-		)
-		(stroke
-			(width 0)
-			(type default)
-		)
-	)
-	(wire
-		(pts
-			(xy 114.3 96.52) (xy 135.89 96.52)
+			(xy 104.14 96.52) (xy 135.89 96.52)
 		)
 		(stroke
@@
 		(pts
 			(xy 135.89 88.9) (xy 132.08 88.9)
-		)
-		(stroke
-			(width 0)
-			(type default)
-		)
-	)
-	(wire
-		(pts
-			(xy 116.84 100.33) (xy 116.84 99.06)
 		)
 		(stroke
@@
 	(hierarchical_label "STP"
 		(shape input)
-		(at 114.3 96.52 180)
+		(at 104.14 96.52 180)
 		(effects
 			(font
@@
 	(hierarchical_label "DIR"
 		(shape input)
-		(at 114.3 100.33 180)
-		(effects
-			(font
+		(at 104.14 99.06 180)
+		(effects
+			(font
